File: 2.0/Hygrometer_2.0.kicad_sch (KiCad schematic)
At the start: 60 parts, among them J1 POWER, J2 DHT11, Q1 Q_NPN_BEC, Q2 Q_NPN_BEC, SW1 WAKE UP, U1 74HC595, U2 ATtiny45V-10P, U3 74HC595

Commit message: Updated resistors for LEDs
Parts:
- R1, R11, R12, R13, R14, R15, R16, R17, R2, R3, R4, R5, R6, R7: value 270 -> 100
Changed lines of the file:
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@@
     (in_bom yes) (on_board yes)
     (property "Reference" "R1" (id 0) (at 120.015 44.45 90))
-    (property "Value" "270" (id 1) (at 130.175 44.45 90))
+    (property "Value" "100" (id 1) (at 130.175 44.45 90))
     (property "Footprint" "Resistor_SMD:R_1206_3216Metric_Pad1.30x1.75mm_HandSolder" (id 2) (at 125.095 43.942 90)
       (effects (font (size 1.27 1.27)) hide)
@@
     (in_bom yes) (on_board yes)
     (property "Reference" "R2" (id 0) (at 120.015 46.99 90))
-    (property "Value" "270" (id 1) (at 130.175 46.99 90))
+    (property "Value" "100" (id 1) (at 130.175 46.99 90))
     (property "Footprint" "Resistor_SMD:R_1206_3216Metric_Pad1.30x1.75mm_HandSolder" (id 2) (at 125.095 46.482 90)
       (effects (font (size 1.27 1.27)) hide)
@@
     (in_bom yes) (on_board yes)
     (property "Reference" "R3" (id 0) (at 120.015 49.53 90))
-    (property "Value" "270" (id 1) (at 130.175 49.53 90))
+    (property "Value" "100" (id 1) (at 130.175 49.53 90))
     (property "Footprint" "Resistor_SMD:R_1206_3216Metric_Pad1.30x1.75mm_HandSolder" (id 2) (at 125.095 49.022 90)
       (effects (font (size 1.27 1.27)) hide)
@@
     (in_bom yes) (on_board yes)
     (property "Reference" "R4" (id 0) (at 120.015 52.07 90))
-    (property "Value" "270" (id 1) (at 130.175 52.07 90))
+    (property "Value" "100" (id 1) (at 130.175 52.07 90))
     (property "Footprint" "Resistor_SMD:R_1206_3216Metric_Pad1.30x1.75mm_HandSolder" (id 2) (at 125.095 51.562 90)
       (effects (font (size 1.27 1.27)) hide)
@@
     (in_bom yes) (on_board yes)
     (property "Reference" "R5" (id 0) (at 120.015 54.61 90))
-    (property "Value" "270" (id 1) (at 130.175 54.61 90))
+    (property "Value" "100" (id 1) (at 130.175 54.61 90))
     (property "Footprint" "Resistor_SMD:R_1206_3216Metric_Pad1.30x1.75mm_HandSolder" (id 2) (at 125.095 54.102 90)
       (effects (font (size 1.27 1.27)) hide)
@@
     (in_bom yes) (on_board yes)
     (property "Reference" "R6" (id 0) (at 120.015 57.15 90))
-    (property "Value" "270" (id 1) (at 130.175 57.15 90))
+    (property "Value" "100" (id 1) (at 130.175 57.15 90))
     (property "Footprint" "Resistor_SMD:R_1206_3216Metric_Pad1.30x1.75mm_HandSolder" (id 2) (at 125.095 56.642 90)
       (effects (font (size 1.27 1.27)) hide)
@@
     (in_bom yes) (on_board yes)
     (property "Reference" "R7" (id 0) (at 120.015 59.69 90))
-    (property "Value" "270" (id 1) (at 130.175 59.69 90))
+    (property "Value" "100" (id 1) (at 130.175 59.69 90))
     (property "Footprint" "Resistor_SMD:R_1206_3216Metric_Pad1.30x1.75mm_HandSolder" (id 2) (at 125.095 59.182 90)
       (effects (font (size 1.27 1.27)) hide)
@@
   )
   (symbol (lib_id "Device:R") (at 125.095 93.98 270) (unit 1)
-    (in_bom yes) (on_board yes) (fields_autoplaced)
+    (in_bom yes) (on_board yes)
     (property "Reference" "R11" (id 0) (at 120.015 92.71 90))
-    (property "Value" "270" (id 1) (at 130.175 92.71 90))
+    (property "Value" "100" (id 1) (at 130.175 92.71 90))
     (property "Footprint" "Resistor_SMD:R_1206_3216Metric_Pad1.30x1.75mm_HandSolder" (id 2) (at 125.095 92.202 90)
       (effects (font (size 1.27 1.27)) hide)
@@
   )
   (symbol (lib_id "Device:R") (at 125.095 96.52 270) (unit 1)
-    (in_bom yes) (on_board yes) (fields_autoplaced)
+    (in_bom yes) (on_board yes)
     (property "Reference" "R12" (id 0) (at 120.015 95.25 90))
-    (property "Value" "270" (id 1) (at 130.175 95.25 90))
+    (property "Value" "100" (id 1) (at 130.175 95.25 90))
     (property "Footprint" "Resistor_SMD:R_1206_3216Metric_Pad1.30x1.75mm_HandSolder" (id 2) (at 125.095 94.742 90)
       (effects (font (size 1.27 1.27)) hide)
@@
     (in_bom yes) (on_board yes)
     (property "Reference" "R13" (id 0) (at 120.015 97.79 90))
-    (property "Value" "270" (id 1) (at 130.175 97.79 90))
+    (property "Value" "100" (id 1) (at 130.175 97.79 90))
     (property "Footprint" "Resistor_SMD:R_1206_3216Metric_Pad1.30x1.75mm_HandSolder" (id 2) (at 125.095 97.282 90)
       (effects (font (size 1.27 1.27)) hide)
@@
     (in_bom yes) (on_board yes)
     (property "Reference" "R14" (id 0) (at 120.015 100.33 90))
-    (property "Value" "270" (id 1) (at 130.175 100.33 90))
+    (property "Value" "100" (id 1) (at 130.175 100.33 90))
     (property "Footprint" "Resistor_SMD:R_1206_3216Metric_Pad1.30x1.75mm_HandSolder" (id 2) (at 125.095 99.822 90)
       (effects (font (size 1.27 1.27)) hide)
@@
     (in_bom yes) (on_board yes)
     (property "Reference" "R15" (id 0) (at 120.015 102.87 90))
-    (property "Value" "270" (id 1) (at 130.175 102.87 90))
+    (property "Value" "100" (id 1) (at 130.175 102.87 90))
     (property "Footprint" "Resistor_SMD:R_1206_3216Metric_Pad1.30x1.75mm_HandSolder" (id 2) (at 125.095 102.362 90)
       (effects (font (size 1.27 1.27)) hide)
@@
     (in_bom yes) (on_board yes)
     (property "Reference" "R16" (id 0) (at 120.015 105.41 90))
-    (property "Value" "270" (id 1) (at 130.175 105.41 90))
+    (property "Value" "100" (id 1) (at 130.175 105.41 90))
     (property "Footprint" "Resistor_SMD:R_1206_3216Metric_Pad1.30x1.75mm_HandSolder" (id 2) (at 125.095 104.902 90)
       (effects (font (size 1.27 1.27)) hide)
@@
     (in_bom yes) (on_board yes)
     (property "Reference" "R17" (id 0) (at 120.015 107.95 90))
-    (property "Value" "270" (id 1) (at 130.175 107.95 90))
+    (property "Value" "100" (id 1) (at 130.175 107.95 90))
     (property "Footprint" "Resistor_SMD:R_1206_3216Metric_Pad1.30x1.75mm_HandSolder" (id 2) (at 125.095 107.442 90)
       (effects (font (size 1.27 1.27)) hide)
@@
     )
     (path "/00000000-0000-0000-0000-00006181d922"
-      (reference "R1") (unit 1) (value "270") (footprint "Resistor_SMD:R_1206_3216Metric_Pad1.30x1.75mm_HandSolder")
+      (reference "R1") (unit 1) (value "100") (footprint "Resistor_SMD:R_1206_3216Metric_Pad1.30x1.75mm_HandSolder")
     )
     (path "/00000000-0000-0000-0000-0000618c9617"
-      (reference "R2") (unit 1) (value "270") (footprint "Resistor_SMD:R_1206_3216Metric_Pad1.30x1.75mm_HandSolder")
+      (reference "R2") (unit 1) (value "100") (footprint "Resistor_SMD:R_1206_3216Metric_Pad1.30x1.75mm_HandSolder")
     )
     (path "/00000000-0000-0000-0000-0000618ca3f9"
-      (reference "R3") (unit 1) (value "270") (footprint "Resistor_SMD:R_1206_3216Metric_Pad1.30x1.75mm_HandSolder")
+      (reference "R3") (unit 1) (value "100") (footprint "Resistor_SMD:R_1206_3216Metric_Pad1.30x1.75mm_HandSolder")
     )
     (path "/00000000-0000-0000-0000-0000618ca3ff"
-      (reference "R4") (unit 1) (value "270") (footprint "Resistor_SMD:R_1206_3216Metric_Pad1.30x1.75mm_HandSolder")
+      (reference "R4") (unit 1) (value "100") (footprint "Resistor_SMD:R_1206_3216Metric_Pad1.30x1.75mm_HandSolder")
     )
     (path "/00000000-0000-0000-0000-0000618cc89e"
-      (reference "R5") (unit 1) (value "270") (footprint "Resistor_SMD:R_1206_3216Metric_Pad1.30x1.75mm_HandSolder")
+      (reference "R5") (unit 1) (value "100") (footprint "Resistor_SMD:R_1206_3216Metric_Pad1.30x1.75mm_HandSolder")
     )
     (path "/00000000-0000-0000-0000-0000618cc8a4"
-      (reference "R6") (unit 1) (value "270") (footprint "Resistor_SMD:R_1206_3216Metric_Pad1.30x1.75mm_HandSolder")
+      (reference "R6") (unit 1) (value "100") (footprint "Resistor_SMD:R_1206_3216Metric_Pad1.30x1.75mm_HandSolder")
     )
     (path "/00000000-0000-0000-0000-0000618cc8aa"
-      (reference "R7") (unit 1) (value "270") (footprint "Resistor_SMD:R_1206_3216Metric_Pad1.30x1.75mm_HandSolder")
+      (reference "R7") (unit 1) (value "100") (footprint "Resistor_SMD:R_1206_3216Metric_Pad1.30x1.75mm_HandSolder")
     )
     (path "/00000000-0000-0000-0000-0000618cc8b0"
@@
     )
     (path "/00000000-0000-0000-0000-0000618d3628"
-      (reference "R11") (unit 1) (value "270") (footprint "Resistor_SMD:R_1206_3216Metric_Pad1.30x1.75mm_HandSolder")
+      (reference "R11") (unit 1) (value "100") (footprint "Resistor_SMD:R_1206_3216Metric_Pad1.30x1.75mm_HandSolder")
     )
     (path "/00000000-0000-0000-0000-0000618d362e"
-      (reference "R12") (unit 1) (value "270") (footprint "Resistor_SMD:R_1206_3216Metric_Pad1.30x1.75mm_HandSolder")
+      (reference "R12") (unit 1) (value "100") (footprint "Resistor_SMD:R_1206_3216Metric_Pad1.30x1.75mm_HandSolder")
     )
     (path "/00000000-0000-0000-0000-0000618d3634"
-      (reference "R13") (unit 1) (value "270") (footprint "Resistor_SMD:R_1206_3216Metric_Pad1.30x1.75mm_HandSolder")
+      (reference "R13") (unit 1) (value "100") (footprint "Resistor_SMD:R_1206_3216Metric_Pad1.30x1.75mm_HandSolder")
     )
     (path "/00000000-0000-0000-0000-0000618d363a"
-      (reference "R14") (unit 1) (value "270") (footprint "Resistor_SMD:R_1206_3216Metric_Pad1.30x1.75mm_HandSolder")
+      (reference "R14") (unit 1) (value "100") (footprint "Resistor_SMD:R_1206_3216Metric_Pad1.30x1.75mm_HandSolder")
     )
     (path "/00000000-0000-0000-0000-0000618d3640"
-      (reference "R15") (unit 1) (value "270") (footprint "Resistor_SMD:R_1206_3216Metric_Pad1.30x1.75mm_HandSolder")
+      (reference "R15") (unit 1) (value "100") (footprint "Resistor_SMD:R_1206_3216Metric_Pad1.30x1.75mm_HandSolder")
     )
     (path "/00000000-0000-0000-0000-0000618d3646"
-      (reference "R16") (unit 1) (value "270") (footprint "Resistor_SMD:R_1206_3216Metric_Pad1.30x1.75mm_HandSolder")
+      (reference "R16") (unit 1) (value "100") (footprint "Resistor_SMD:R_1206_3216Metric_Pad1.30x1.75mm_HandSolder")
     )
     (path "/00000000-0000-0000-0000-0000618d364c"
-      (reference "R17") (unit 1) (value "270") (footprint "Resistor_SMD:R_1206_3216Metric_Pad1.30x1.75mm_HandSolder")
+      (reference "R17") (unit 1) (value "100") (footprint "Resistor_SMD:R_1206_3216Metric_Pad1.30x1.75mm_HandSolder")
     )
     (path "/00000000-0000-0000-0000-0000618d3652"
